Commit message: update car2 package

File: car2/urdf/car2.urdf (robot description, URDF)
Before this commit: robot car2, 11 links, 10 joints
Joints:
- removed joint castwheel
- removed joint leftwheel
- removed joint rightwheel
- added joint castwheel_joint: type continuous, parent base_link, child castwheel, origin xyz=-0.0164468565720474 -0.00527324448375706 -0.025 rpy=1.79986954685685 -0.424347021577185 0.792685410767129, axis 0.578881459990206 -0.0793276054052651 0.811543828945962
- added joint leftwheel_joint: type continuous, parent base_link, child leftwheel, origin xyz=0.055 -0.110423702246605 -0.035 rpy=-1.5707963267949 -0.105014840444308 3.14159265358979, axis 0 0 1
- added joint rightwheel_joint: type continuous, parent base_link, child rightwheel, origin xyz=0.055 0.110423702246602 -0.035 rpy=1.5707963267949 -0.261061307663736 0, axis 0 0 1
- joint fin1: limit lower=0 upper=0.05 effort=0 velocity=1.01 -> lower=-0.05 upper=0 effort=0 velocity=1.01
- joint joint3: limit lower=0 upper=0.26 effort=0 velocity=1.5 -> lower=-0.26 upper=0 effort=0 velocity=1.5

Commit message: urdf edition 2

File: car2/urdf/car2.urdf (robot description, URDF)
Before this commit: robot car2, 11 links, 10 joints
Links:
- link base_link: mass 30.028 -> 10.1
